Commit message: fix bug localization

File: src/ttbot_description/urdf/ttbot.urdf.xacro (robot description, xacro)
@@ -1,17 +1,13 @@
 <?xml version="1.0"?>
 <robot name="ttbot" xmlns:xacro="http://www.ros.org/wiki/xacro">
-  <!-- Arg dùng cho Gazebo / Ignition -->
   <xacro:arg name="is_ignition" default="true"/>
-  <!-- =============== INCLUDE GAZEBO =============== -->
   <xacro:include filename="$(find ttbot_description)/urdf/ttbot_gazebo.xacro" />
-  <!-- ================= CONSTANTS ================= -->
-  <xacro:property name="wheel_radius" value="0.15"/>        <!-- bán kính bánh xe -->
-  <xacro:property name="wheel_width"  value="0.06"/>        <!-- bề dày bánh -->
-  <xacro:property name="wheelbase"    value="0.65"/>         <!-- khoảng cách giữa 2 trục -->
-  <xacro:property name="track_width"  value="0.55"/>        <!-- khoảng cách 2 bánh cùng trục -->
-  <xacro:property name="chassis_length" value="1.0"/>       <!-- chiều dài thân -->
-  <xacro:property name="chassis_width"  value="0.6"/>       <!-- chiều rộng thân -->
-  <xacro:property name="chassis_height" value="0.45"/>      <!-- chiều cao thân -->
-  <!-- ================= HELPER MACROS ================= -->
+  <xacro:property name="wheel_radius" value="0.15"/>
+  <xacro:property name="wheel_width"  value="0.06"/>
+  <xacro:property name="wheelbase"    value="0.65"/>
+  <xacro:property name="track_width"  value="0.55"/>
+  <xacro:property name="chassis_length" value="1.0"/>
+  <xacro:property name="chassis_width"  value="0.6"/>
+  <xacro:property name="chassis_height" value="0.45"/>
   <xacro:macro name="inertial_cyl" params="mass r l">
     <inertial>
@@ -24,16 +20,12 @@
     </inertial>
   </xacro:macro>
-  <!-- ================= BASE LINK ================= -->
   <link name="base_link">
-    <!-- Thân chính (visual) -->
     <visual>
       <geometry>
         <box size="${chassis_length} ${chassis_width} ${chassis_height}"/>
       </geometry>
-      <!-- thân trên mặt đất -->
       <origin xyz="0 0 ${wheel_radius + 0.5 * chassis_height}" rpy="0 0 0"/>
       <material name="red"><color rgba="0.8 0.1 0.1 1.0"/></material>
     </visual>
-    <!-- Mui xe -->
     <visual>
       <origin xyz="0 0 ${wheel_radius + chassis_height}" rpy="0 0 0"/>
@@ -41,5 +33,4 @@
       <material name="darkred"><color rgba="0.8 0.1 0.1 1.0"/></material>
     </visual>
-    <!-- Gương hai bên -->
     <visual>
       <origin xyz="0.4 ${0.5*chassis_width + 0.05} ${wheel_radius + chassis_height}"/>
@@ -52,5 +43,4 @@
       <material name="gray"><color rgba="0.5 0.5 0.5 1"/></material>
     </visual>
-    <!-- Đèn pha -->
     <visual>
       <origin xyz="${0.5*chassis_length + 0.03} ${0.25*chassis_width} ${wheel_radius + 0.6*chassis_height}"/>
@@ -63,5 +53,4 @@
       <material name="white"><color rgba="1 1 1 1"/></material>
     </visual>
-    <!-- COLLISION thân -->
     <collision>
       <origin xyz="0 0 ${wheel_radius + 0.5 * chassis_height}" rpy="0 0 0"/>
@@ -70,5 +59,4 @@
       </geometry>
     </collision>
-    <!-- INERTIAL thân -->
     <inertial>
       <origin xyz="0 0 ${wheel_radius + 0.5 * chassis_height}" rpy="0 0 0"/>
@@ -81,5 +69,4 @@
     </inertial>
   </link>
-  <!-- ================= WHEEL MACRO ================= -->
   <xacro:macro name="wheel_link" params="name">
     <link name="${name}">
@@ -96,7 +83,4 @@
     </link>
   </xacro:macro>
-  <!-- ================= WHEEL + STEERING LINKS ================= -->
-  <!-- Link trung gian cho lái -->
-  <!-- Link trung gian cho lái - phải có collision + inertial -->
   <link name="front_left_steering_link">
     <collision>
@@ -129,5 +113,4 @@
     </inertial>
   </link>
-  <!-- Bánh -->
   <xacro:wheel_link name="front_left_wheel"/>
   <xacro:wheel_link name="front_right_wheel"/>
@@ -135,5 +118,4 @@
   <xacro:wheel_link name="rear_right_wheel"/>
   <!-- ================= JOINTS ================= -->
-  <!-- FRONT STEERING JOINTS (Ackermann) -->
   <joint name="front_left_steering_joint" type="revolute">
     <parent link="base_link"/>
@@ -151,5 +133,4 @@
     <mimic joint="front_left_steering_joint" multiplier="1.0"/>
   </joint>
-  <!-- STEERING_LINK -> WHEEL : quay bánh quanh trục Y -->
   <joint name="front_left_wheel_joint" type="continuous">
     <parent link="front_left_steering_link"/>
@@ -164,5 +145,4 @@
     <axis xyz="0 1 0"/>
   </joint>
-  <!-- REAR DRIVE JOINTS (motor) -->
   <joint name="rear_left_wheel_joint" type="continuous">
     <parent link="base_link"/>
@@ -179,9 +159,7 @@
   <!-- ================= IMU LINK ================= -->
   <link name="imu_link">
-    <!-- Hình trụ nhỏ giống tụ/IMU -->
-    <visual>
-      <origin xyz="0 0 0" rpy="0 0 0"/>
-      <geometry>
-        <!-- Bán kính ~3cm, cao ~6cm -->
+    <visual>
+      <origin xyz="0 0 0" rpy="0 0 0"/>
+      <geometry>
         <cylinder radius="0.04" length="0.05"/>
       </geometry>
@@ -205,14 +183,7 @@
   </link>
   <!-- ================= IMU JOINT ================= -->
-  <!-- Đặt IMU trên nóc xe, ngay chính giữa -->
   <joint name="imu_joint" type="fixed">
     <parent link="base_link"/>
     <child link="imu_link"/>
-    <!--
-      wheel_radius = 0.15
-      chassis_height = 0.25
-      Nóc (mui) ~ wheel_radius + chassis_height + 0.1 = 0.5
-      Đặt tâm IMU nhô lên thêm ~3cm: +0.13
-    -->
     <origin xyz="0 0 ${wheel_radius + chassis_height + 0.13}" rpy="0 0 0"/>
     <axis xyz="0 0 0"/>
@@ -220,13 +191,11 @@
   <!-- ================= GPS LINK ================= -->
   <link name="gps_link">
-    <!-- Hình trụ nhỏ màu đen -->
-    <visual>
-      <origin xyz="0 0 0" rpy="0 0 0"/>
-      <geometry>
-        <!-- Bán kính / chiều cao tương tự IMU -->
+    <visual>
+      <origin xyz="0 0 0" rpy="0 0 0"/>
+      <geometry>
         <cylinder radius="0.04" length="0.05"/>
       </geometry>
       <material name="gps_black">
-        <color rgba="0 0 0 1"/> <!-- Màu đen -->
+        <color rgba="0 0 0 1"/>
       </material>
     </visual>
@@ -246,13 +215,7 @@
   </link>
   <!-- ================= GPS JOINT ================= -->
-  <!-- Đặt GPS trên nóc xe, lệch nhẹ về phía trước so với IMU -->
   <joint name="gps_joint" type="fixed">
     <parent link="base_link"/>
     <child link="gps_link"/>
-    <!--
-      IMU đang dùng:
-        z = wheel_radius + chassis_height + 0.13
-      GPS: cùng độ cao, lệch trục x về phía trước 10cm
-    -->
     <origin xyz="0.1 0 ${wheel_radius + chassis_height + 0.13}" rpy="0 0 0"/>
     <axis xyz="0 0 0"/>
@@ -268,5 +231,4 @@
       </xacro:unless>
     </hardware>
-    <!-- Bánh sau: điều khiển velocity -->
     <joint name="rear_left_wheel_joint">
       <command_interface name="velocity"/>
@@ -279,5 +241,4 @@
       <state_interface name="velocity"/>
     </joint>
-    <!-- Góc lái: điều khiển position -->
     <joint name="front_left_steering_joint">
       <command_interface name="position"/>
@@ -291,5 +252,4 @@
     </joint>
   </ros2_control>
-  <!-- ================= GAZEBO MACRO ================= -->
   <xacro:ttbot_gazebo/>
 </robot>

File: src/ttbot_description/urdf/ttbot_gazebo.xacro (robot description, xacro)
@@ -1,12 +1,5 @@
 <?xml version="1.0"?>
 <robot xmlns:xacro="http://www.ros.org/wiki/xacro">
-  <!--
-    Macro: ttbot_gazebo
-    - Thêm thuộc tính ma sát cho 4 bánh
-    - Thêm plugin ros2_control cho Ignition / Gazebo Sim
-    - Dùng chung biến is_ignition được khai báo bằng <xacro:arg> trong file ttbot.urdf.xacro
-  -->
   <xacro:macro name="ttbot_gazebo" params="">
-    <!-- Hai bánh sau là bánh chủ động, có ma sát cao -->
     <gazebo reference="rear_left_wheel">
       <mu1>1000000.0</mu1>    <!-- ma sát dọc -->
@@ -27,5 +20,4 @@
       <fdir1>1 0 0</fdir1>
     </gazebo>
-    <!-- Hai bánh trước có ma sát thấp hơn để dễ lái -->
     <gazebo reference="front_left_wheel">
       <mu1>100000.0</mu1>
@@ -44,7 +36,5 @@
       <maxVel>0.1</maxVel>
     </gazebo>
-    <!-- ROS 2 Control plugin cho Ignition / Gazebo Sim -->
     <gazebo>
-      <!-- ROS 2 Humble dùng Ignition / Gazebo Fortress -->
       <xacro:if value="$(arg is_ignition)">
         <plugin filename="ign_ros2_control-system"
@@ -55,5 +45,4 @@
         </plugin>
       </xacro:if>
-      <!-- ROS 2 Iron trở lên dùng Gazebo Sim (gz) -->
       <xacro:unless value="$(arg is_ignition)">
         <plugin filename="gz_ros2_control-system"
@@ -65,5 +54,4 @@
       </xacro:unless>
     </gazebo>
-  <!-- IMU -->
   <gazebo reference="imu_link">
     <sensor name="imu" type="imu">

File: src/ttbot_description/urdf/ttbot_ros2_control.xacro (robot description, xacro)
@@ -1,11 +1,5 @@
 <?xml version="1.0"?>
 <robot xmlns:xacro="http://www.ros.org/wiki/xacro">
-  <!--
-    Macro: ttbot_gazebo
-    - ma sát, contact cho bánh
-    - plugin ros2_control cho Ignition / Gazebo Sim
-  -->
   <xacro:macro name="ttbot_gazebo" params="">
-    <!-- Hai bánh sau: ma sát cao hơn một chút -->
     <gazebo reference="rear_left_wheel">
       <mu1>2.0</mu1>
@@ -24,5 +18,4 @@
       <maxVel>0.5</maxVel>
     </gazebo>
-    <!-- Hai bánh trước -->
     <gazebo reference="front_left_wheel">
       <mu1>1.5</mu1>
@@ -41,7 +34,5 @@
       <maxVel>0.5</maxVel>
     </gazebo>
-    <!-- Plugin ROS 2 Control -->
     <gazebo>
-      <!-- ROS 2 Humble + Ignition (Fortress, Garden...) -->
       <xacro:if value="$(arg is_ignition)">
         <plugin filename="ign_ros2_control-system"
@@ -50,5 +41,4 @@
         </plugin>
       </xacro:if>
-      <!-- ROS 2 Iron+ + Gazebo Sim (gz) -->
       <xacro:unless value="$(arg is_ignition)">
         <plugin filename="gz_ros2_control-system"
